Commit message: Model the team's Unitree L1 at its real mount, the robot body as an occluder, and wheel ruts
- uic_bot_2027.xacro: the 3D LiDAR is the team's Unitree L1 at the comp-day-one mount (-0.353, 0, 0.721) from
  base_link, upside down (EDT-Lunabotics-2026 branch comp-day-one, test.launch.py static transform).
- sensors.py: L1-like scan (l1_dirs; 11 Hz core, 180 Hz mirror, 21600 points/s, from the L1 manual), any mount
  rotation, the robot's own body blocking and returning rays (robot.BodyCaster, Embree when installed), and an
  extrinsic calibration error option. Earlier cases are unchanged: seed 3000 reproduces results_rob/base exactly.
- ruts.py: wheel ruts stamped into the arena height field, 3.2 cm deep from Wong 2012 Eq. (6) with Lunar Sourcebook
  soil values (not BP-1), plus berms; earlier trips weave through the obstacle zone.
- params.py: L1 profile, ROBOT and RUTS tables with sources.

Co-Authored-By: Claude Opus 5.5 (1M context) <noreply@anthropic.com>
Claude-Session: https://claude.ai/code/session_01DhdYww2ugdyJGkGRKdFNKq

File: sim/robot/uic_bot_2027.xacro (robot description, xacro)
@@ -4,7 +4,10 @@
   src/description_pkg/urdf/uic_bot.xacro at commit a720e46 (2026 robot). Body, wheels, D456 and IMU are unchanged.
   Changes for the 2027 autonomy plan (each one Assumed until the team measures the real robot):
-  - lidar3d_link: a generic 3D LiDAR replaces the 2D RPLIDAR S3, at the S3's mount (0, 0.102, 0.470), pitched 30 deg
-    down. Housing is a generic 0.05 m radius x 0.07 m cylinder. Gazebo sensor: 16 beams over +-15 deg, 0.4 deg steps
-    (the sandbox "spin16" pattern), 0.3 to 8 m.
+  - lidar3d_link: the team's 3D LiDAR, a Unitree L1 (branches 5-27-2026 and comp-day-one: unitree_lidar_ros2 driver,
+    unilidar_sdk, Point-LIO config unilidar_l1.yaml), replacing the 2D RPLIDAR S3. Mount copied from comp-day-one
+    (3bd79d3) src/neptune_bringup/launch/test.launch.py, static transform base_link -> s3_lidar_link:
+    xyz (-0.353, 0, 0.721), roll 180 deg ("upside down"), so its 360 x 90 deg hemisphere looks down. Housing is the
+    L1's 75 x 75 x 65 mm (Unitree L1 user manual v1.1). Gazebo sensor: a 360 x 90 deg approximation of its field of
+    view; the sandbox models the L1's mirror-and-core scan itself (sensors.l1_dirs).
   - d455_link: moved from the rear (facing back) to the front centre, pitched 40 deg down (Angelo's 2027 layout;
     the 40 deg is Angelo's, the position is Assumed).
@@ -89,5 +92,5 @@
     <visual>
       <geometry>
-        <cylinder radius="0.05" length="0.07" />
+        <box size="0.075 0.075 0.065" />
       </geometry>
       <origin xyz="0 0 0" rpy="0 0 0" />
@@ -96,5 +99,5 @@
     <collision>
       <geometry>
-        <cylinder radius="0.05" length="0.07" />
+        <box size="0.075 0.075 0.065" />
       </geometry>
       <origin xyz="0 0 0" rpy="0 0 0" />
@@ -225,5 +228,5 @@
     <parent link="base_link" />
     <child link="lidar3d_link" />
-    <origin xyz="0.0 0.102 0.470" rpy="0 0.5236 0" />
+    <origin xyz="-0.353 0 0.721" rpy="3.14159 0 0" />
   </joint>
   <joint name="base_rear_cam_joint" type="fixed">
@@ -453,23 +456,23 @@
         <pose>0 0 0 0 0 0</pose>
         <visualize>false</visualize>
-        <update_rate>10.0</update_rate>
+        <update_rate>11.0</update_rate>
         <ray>
           <scan>
             <horizontal>
-              <samples>900</samples>
+              <samples>360</samples>
               <resolution>1</resolution>
               <min_angle>-3.14159</min_angle>
-              <max_angle>3.13461</max_angle>
+              <max_angle>3.12414</max_angle>
             </horizontal>
             <vertical>
-              <samples>16</samples>
+              <samples>60</samples>
               <resolution>1</resolution>
-              <min_angle>-0.2618</min_angle>
-              <max_angle>0.2618</max_angle>
+              <min_angle>0.0</min_angle>
+              <max_angle>1.5708</max_angle>
             </vertical>
           </scan>
           <range>
-            <min>0.3</min>
-            <max>8.0</max>
+            <min>0.05</min>
+            <max>15.0</max>
           </range>
           <noise>

Commit message: Move the L1 to the front top, 45 deg down, in the 2027 robot model
Angelo chose the front mount after the hazard and localization runs. robot.LIDAR_MOUNTS
keeps the team's 2026 rear mount as rear2026; run_selfmask.sh and localize.py name it, so
the older runs reproduce exactly (checked on seed 3000 and on all 1920 localization rows).

Co-Authored-By: Claude Opus 5.5 (1M context) <noreply@anthropic.com>
Claude-Session: https://claude.ai/code/session_01DhdYww2ugdyJGkGRKdFNKq

File: sim/robot/uic_bot_2027.xacro (robot description, xacro)
@@ -5,7 +5,10 @@
   Changes for the 2027 autonomy plan (each one Assumed until the team measures the real robot):
   - lidar3d_link: the team's 3D LiDAR, a Unitree L1 (branches 5-27-2026 and comp-day-one: unitree_lidar_ros2 driver,
-    unilidar_sdk, Point-LIO config unilidar_l1.yaml), replacing the 2D RPLIDAR S3. Mount copied from comp-day-one
-    (3bd79d3) src/neptune_bringup/launch/test.launch.py, static transform base_link -> s3_lidar_link:
-    xyz (-0.353, 0, 0.721), roll 180 deg ("upside down"), so its 360 x 90 deg hemisphere looks down. Housing is the
+    unilidar_sdk, Point-LIO config unilidar_l1.yaml), replacing the 2D RPLIDAR S3. Since 2026-10-12 it sits at the
+    front top, upside down and pitched so its axis points 45 deg forward of straight down: xyz (0.45, 0, 0.4849),
+    rpy (180, -45, 0) deg, 0.75 m above the ground (Angelo's choice after the sandbox hazard and localization runs;
+    the position is Assumed until the team finds a real mount point there). The team's 2026 mount, from comp-day-one
+    (3bd79d3) src/neptune_bringup/launch/test.launch.py, static transform base_link -> s3_lidar_link, was
+    xyz (-0.353, 0, 0.721), roll 180 deg ("upside down"); robot.LIDAR_MOUNTS["rear2026"] keeps it. Housing is the
     L1's 75 x 75 x 65 mm (Unitree L1 user manual v1.1). Gazebo sensor: a 360 x 90 deg approximation of its field of
     view; the sandbox models the L1's mirror-and-core scan itself (sensors.l1_dirs).
@@ -228,5 +231,5 @@
     <parent link="base_link" />
     <child link="lidar3d_link" />
-    <origin xyz="-0.353 0 0.721" rpy="3.14159 0 0" />
+    <origin xyz="0.45 0 0.4849" rpy="3.14159 -0.785398 0" />
   </joint>
   <joint name="base_rear_cam_joint" type="fixed">
